File: rcdecade.sch (KiCad schematic (older format))
At the start: 114 parts, among them SW1 SW_Rotary10, SW10 SW_RotaryBCD, SW11 SW_RotaryBCD, SW12 SW_Rotary10, SW13 SW_Rotary10, SW2 SW_RotaryBCD, SW3 SW_RotaryBCD, SW4 SW_Rotary10, SW5 SW_RotaryBCD, SW6 SW_Rotary10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

Commit message: R Decade only
Parts:
- removed C1: 100p, Capacitor_SMD:C_0805_2012Metric, symbol Device:C
- removed C10, C8, C9: 2n, Capacitor_SMD:C_0805_2012Metric, symbol Device:C
- removed C11: 3.3n, Capacitor_SMD:C_0805_2012Metric, symbol Device:C
- removed C12: 4.7n, Capacitor_SMD:C_0805_2012Metric, symbol Device:C
- removed C13: 10n, Capacitor_SMD:C_0805_2012Metric, symbol Device:C
- removed C14, C15, C16: 20n, Capacitor_SMD:C_0805_2012Metric, symbol Device:C
- removed C17: 33nF, Capacitor_SMD:C_0805_2012Metric, symbol Device:C
- removed C18: 47nF, Capacitor_SMD:C_0805_2012Metric, symbol Device:C
- removed C19: 100n, Capacitor_SMD:C_0805_2012Metric, symbol Device:C
- removed C2, C3, C4: 200p, Capacitor_SMD:C_0805_2012Metric, symbol Device:C
- removed C20, C21, C22: 200n, Capacitor_SMD:C_0805_2012Metric, symbol Device:C
- removed C23: 330n, Capacitor_SMD:C_0805_2012Metric, symbol Device:C
- removed C24: 470n, Capacitor_SMD:C_0805_2012Metric, symbol Device:C
- removed C25, C26, C27: 1u, Capacitor_SMD:C_0805_2012Metric, symbol Device:C
- removed C28: 1.8u, Capacitor_SMD:C_0805_2012Metric, symbol Device:C
- removed C29: 2.2u, Capacitor_SMD:C_0805_2012Metric, symbol Device:C
- removed C30: 3.3u, Capacitor_SMD:C_0805_2012Metric, symbol Device:C
- removed C31: 4.7u, Capacitor_SMD:C_0805_2012Metric, symbol Device:C
- removed C32: 10u, Capacitor_SMD:C_0805_2012Metric, symbol Device:C
- removed C33, C34, C35: 20u, Capacitor_SMD:C_0805_2012Metric, symbol Device:C
- removed C36: 33u, Capacitor_SMD:C_0805_2012Metric, symbol Device:C
- removed C37: 47u, Capacitor_SMD:C_0805_2012Metric, symbol Device:C
- removed C5: 330p, Capacitor_SMD:C_0805_2012Metric, symbol Device:C
- removed C6: 470p, Capacitor_SMD:C_0805_2012Metric, symbol Device:C
- removed C7: 1n, Capacitor_SMD:C_0805_2012Metric, symbol Device:C
- removed S1: JS202011SCQN, digikey-footprints:Switch_Slide_JS202011SCQN, symbol dk_Slide-Switches:JS202011SCQN
- removed SW10, SW11, SW2, SW3, SW5, SW7: SW_RotaryBCD, thumbwheel:Switch_Thumbwheel_BCD, symbol w6ipa_switch:SW_RotaryBCD
- added J1, J2: Conn_01x01_Female, Connector_Wire:SolderWirePad_1x01_Drill2mm, symbol Connector:Conn_01x01_Female
- added LOGO1: dahu-logo, w6ipa-footprints:W6IPA-Logo-9mmx8mm, symbol w6ipa_graphic:dahu-logo
Connections:
- net RCommon: now also J2.1 (Pin_1)
- net 2 renamed Resistances
- net Resistances: now also J1.1 (Pin_1)
Other:
- note removed: "x1 nF\n\n"
- note removed: "x1 uF"
- note removed: "x10 nF\n\n"
- note removed: "x10 uF"
- note removed: "x100 nF\n\n"
- note removed: "x100 pF\n"

Commit message: Fix // serial
Connections:
- net RCommon: no longer SW12.C (11), SW13.C (11), SW4.C (11), SW6.C (11), SW8.C (11), SW9.C (11)
- net Resistances: no longer R1.1, R10.1, R19.1, R28.1, R37.1, R46.1, SW1.0 (1), SW12.0 (1), SW4.0 (1), SW6.0 (1), SW8.0 (1), SW9.0 (1)
- new net: R1.1, SW1.0 (1), SW4.C (11)
- new net: R10.1, SW4.0 (1), SW6.C (11)
- new net: R19.1, SW6.0 (1), SW8.C (11)
- new net: R28.1, SW8.0 (1), SW9.C (11)
- new net: R37.1, SW12.C (11), SW9.0 (1)
- new net: R46.1, SW12.0 (1), SW13.C (11)
Other:
- moved on the sheet: J1, J2, R1, R10, R11, R12, R13, R14, R15, R16, R17, R18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
